File: experiments/paul-nanosim-r04/hardware/collar-tracker.kicad_pcb (KiCad board)
At the start: 4 copper layers, 35 x 28 mm, 54 parts, among them J1 LTE antenna / 50R, J2 GNSS antenna / passive, J3 5V charging input, J4 Protected cell + NTC, J5 DIGITAL health sensor interfa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, J6 SIM8051-6-0-14-00-A, J7 SWD / debug, U1 nRF9151-LACA, U2 SKY65943-11, U3 BQ25185DLHR, U4 TPS7A0218PDBVR, U5 LIS2DW12TR

Commit message: wip(pcb): rework charger escapes and retain native routing evidence
Routing:
- net /I2C_SCL: track 38.0 -> 76.2 mm
- net /BAT_NTC: track 1.43 -> 8.65 mm, vias 1 -> 2
- net /VSYS: track 61.3 -> 67.7 mm, vias 5 -> 6
- net /ISET: track 0.00 -> 4.49 mm
- net /VIN_5V: track 3.51 -> 7.85 mm, vias 1 -> 2
- net /ILIM_VSET: track 0.00 -> 3.06 mm
- net /GND: track 83.8 -> 86.8 mm, vias 68 -> 67
- net /VDD_NRF: track 16.0 -> 17.8 mm
- net /VBAT: track 23.8 -> 25.6 mm, vias 2 -> 3
- net /VIO_1V8: track 96.6 -> 98.2 mm
- net /CHG_FAULT: track 11.7 -> 13.2 mm, vias 1 -> 2
